File: circuit/v2b/tail.kicad_pcb (KiCad board)
At the start: 2 copper layers, 40 x 40 mm, 53 parts, among them J1 LED_DEBUG, J11 UART, J19 LiPo, J2 POWER_DEBUG, J25 USB_OTG, J3 LiPo, J9 DEBUG, Q1 Q_NMOS_GSD, SW1 SW_SPDT, U1 DWM1000, U2 EFM32HG222F64, U3 MC3630, U4 XC6215B332NR, U5 MCP73831-2-OT, Y1 32.768kHz CFPX-217 20ppm 7pF

Commit message: circuit: route v2b PCB
Signed-off-by: Gavan Fantom <gavan.fantom@unipart.io>
Parts:
- added Q2: Q_NMOS_GSD, TO_SOT_Packages_SMD:SOT-323_SC-70, F.Cu at (137.6, 98.1)
- added Q3: Q_NMOS_GSD, TO_SOT_Packages_SMD:SOT-323_SC-70, F.Cu at (141.1, 98.1)
- R10: value 2.2K -> 5.1K
- moved R9 3.82 mm to (144.7, 92.2), turned to 0 degrees
- moved C6 3.40 mm to (142.3, 95.8), turned to 0 degrees
- moved C7 3.26 mm to (142.8, 94.2), turned to 0 degrees
- moved C5 1.36 mm to (138.5, 95.8), turned to 180 degrees
- moved C12 0.28 mm to (144.9, 94.3), turned to 270 degrees
Connections:
- J11 pad 1: UART_RX -> UART_RX_HV
- J11 pad 2: UART_TX -> UART_TX_HV
- J25 pad 2: Net-(J25-Pad2) -> UART_TX_HV
- J25 pad 3: Net-(J25-Pad3) -> UART_RX_HV
Routing:
- net UART_TX_HV: track 0.00 -> 36.3 mm, vias 0 -> 3
- net UART_RX_HV: track 0.00 -> 35.4 mm, vias 0 -> 5
- net UART_RX: track 7.97 -> 15.6 mm, vias 1 -> 4
- net ACCEL_PWR: track 80.1 -> 86.9 mm
- net BATT_MON: track 17.7 -> 15.0 mm
- net UART_TX: track 4.34 -> 5.18 mm, vias 1 -> 2
- net ACCEL_SCK: track 22.3 -> 21.7 mm
- net GND: track 115.4 -> 116.0 mm, vias 52 -> 48
Other:
- board text added: "v2b"
- board text removed: "v2a"
